File: buck-converter-breakout-3v3.kicad_pcb (KiCad board)
At the start: 2 copper layers, 19.8 x 45.8 mm, 9 parts, among them J1 Conn_01x01_Pin, J2 Conn_01x02_Pin, J3 Barrel_Jack_Switch, U1 XL1509-3.3

Commit message: DRC
Other:
- board text added: "Designed by Mori Adrian Rosland"
Changed lines of the file:
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@@
 		(property ki_fp_filters "SOIC*3.9x4.9mm*P1.27mm*")
 		(sheetname "/")
-		(sheetfile "emi-test-board.kicad_sch")
+		(sheetfile "buck-converter-breakout-3v3.kicad_sch")
 		(attr smd)
 		(fp_line
@@
 		(property ki_fp_filters "C_*")
 		(sheetname "/")
-		(sheetfile "emi-test-board.kicad_sch")
+		(sheetfile "buck-converter-breakout-3v3.kicad_sch")
 		(attr smd)
 		(fp_line
@@
 		(property ki_fp_filters "C_*")
 		(sheetname "/")
-		(sheetfile "emi-test-board.kicad_sch")
+		(sheetfile "buck-converter-breakout-3v3.kicad_sch")
 		(attr through_hole)
 		(fp_line
@@
 		(property ki_fp_filters "Connector*:*_1x??_*")
 		(sheetname "/")
-		(sheetfile "emi-test-board.kicad_sch")
+		(sheetfile "buck-converter-breakout-3v3.kicad_sch")
 		(attr through_hole)
 		(fp_line
@@
 		(property ki_fp_filters "BarrelJack*")
 		(sheetname "/")
-		(sheetfile "emi-test-board.kicad_sch")
+		(sheetfile "buck-converter-breakout-3v3.kicad_sch")
 		(attr through_hole)
 		(fp_line
@@
 		(property ki_fp_filters "Connector*:*_1x??_*")
 		(sheetname "/")
-		(sheetfile "emi-test-board.kicad_sch")
+		(sheetfile "buck-converter-breakout-3v3.kicad_sch")
 		(attr through_hole)
 		(fp_line
@@
 		(property ki_fp_filters "TO-???* *_Diode_* *SingleDiode* D_*")
 		(sheetname "/")
-		(sheetfile "emi-test-board.kicad_sch")
+		(sheetfile "buck-converter-breakout-3v3.kicad_sch")
 		(attr through_hole)
 		(fp_line
@@
 			(effects
 				(font
-					(size 0.64 0.64)
+					(size 1 1)
 					(thickness 0.15)
 				)
@@
 		(property ki_fp_filters "Choke_* *Coil* Inductor_* L_*")
 		(sheetname "/")
-		(sheetfile "emi-test-board.kicad_sch")
+		(sheetfile "buck-converter-breakout-3v3.kicad_sch")
 		(attr smd)
 		(fp_line
@@
 		(property ki_fp_filters "C_*")
 		(sheetname "/")
-		(sheetfile "emi-test-board.kicad_sch")
+		(sheetfile "buck-converter-breakout-3v3.kicad_sch")
 		(attr through_hole)
 		(fp_line
@@
 		)
 	)
+	(gr_text "Designed by\nMori Adrian Rosland"
+		(at 111.25 50.5 90)
+		(layer "B.SilkS")
+		(effects
+			(font
+				(size 1 1)
+				(thickness 0.15)
+			)
+			(justify left bottom mirror)
+		)
+	)
 	(segment
 		(start 101.25 81.81)
@@
 		(polygon
 			(pts
-				(xy 98.5 78.75) (xy 98.5 78.75) (xy 98.5 75) (xy 98.25 74.75) (xy 95.25 74.75) (xy 95 75) (xy 95 77.75)
-				(xy 95.25 78) (xy 95.5 78) (xy 95.75 78.25) (xy 95.75 80.75) (xy 96 81) (xy 97.75 81) (xy 98 80.75)
-				(xy 98 80) (xy 98.25 79.75) (xy 102 79.75) (xy 102.25 79.5) (xy 102.25 78.75)
+				(xy 98.5 78.75) (xy 98.5 75) (xy 98.25 74.75) (xy 95.25 74.75) (xy 95 75) (xy 95 77.75) (xy 95.25 78)
+				(xy 95.5 78) (xy 95.75 78.25) (xy 95.75 80.75) (xy 96 81) (xy 97.75 81) (xy 98 80.75) (xy 98 80)
+				(xy 98.25 79.75) (xy 102 79.75) (xy 102.25 79.5) (xy 102.25 78.75)
 			)
 		)

Commit message: ignore production files
Parts:
- L1: footprint project_footprints:INDM3225X240N -> Inductor_SMD:L_Chilisin_BMRF00101040
- moved J2 10.6 mm to (102.5, 96.2), turned to 90 degrees
- moved L1 4.95 mm to (93.2, 85.0)
- moved D1 3.81 mm to (93.2, 74.8)
- moved C3 0.92 mm to (102.4, 88.5)
Other:
- board size 19.8 x 45.8 mm -> 25 x 50.5 mm
