File: buck-converter-breakout-3v3.kicad_sch (KiCad schematic)
At the start: 9 parts, among them J1 Conn_01x01_Pin, J2 Conn_01x02_Pin, J3 Barrel_Jack_Switch, U1 XL1509-3.3

Commit message: DRC
Other:
- company: (none) -> Mori Adrian Rosland
- title: (none) -> Buck-converter 3V3 Breakout Board
Changed lines of the file:
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@@
 	(generator_version "9.0")
 	(paper "A4")
+	(title_block
+		(title "Buck-converter 3V3 Breakout Board")
+		(date "2025-10-19")
+		(rev "1.0")
+		(company "Mori Adrian Rosland")
+	)
 	(text "Keep feedback wiring away from inductor flux"
 		(exclude_from_sim no)
@@
 	)
 	(junction
+		(at 179.07 95.25)
+		(diameter 0)
+		(color 0 0 0 0)
+	)
+	(junction
 		(at 87.63 95.25)
 		(diameter 0)
@@
 	(wire
 		(pts
+			(xy 179.07 95.25) (xy 179.07 96.52)
+		)
+		(stroke
+			(width 0)
+			(type default)
+		)
+	)
+	(wire
+		(pts
 			(xy 87.63 102.87) (xy 87.63 106.68)
 		)
@@
 	(wire
 		(pts
-			(xy 163.83 95.25) (xy 170.18 95.25)
+			(xy 163.83 95.25) (xy 179.07 95.25)
 		)
 		(stroke
@@
 	(wire
 		(pts
-			(xy 170.18 95.25) (xy 170.18 93.98)
+			(xy 179.07 95.25) (xy 179.07 93.98)
 		)
 		(stroke
@@
 	)
 	(symbol
+		(lib_id "power:PWR_FLAG")
+		(at 179.07 96.52 180)
+		(unit 1)
+		(exclude_from_sim no)
+		(in_bom yes)
+		(on_board yes)
+		(dnp no)
+		(fields_autoplaced yes)
+		(property "Reference" "#FLG02"
+			(at 179.07 98.425 0)
+			(effects
+				(font
+					(size 1.27 1.27)
+				)
+				(hide yes)
+			)
+		)
+		(property "Value" "PWR_FLAG"
+			(at 179.07 100.33 0)
+			(effects
+				(font
+					(size 0.762 0.762)
+				)
+			)
+		)
+		(property "Footprint" ""
+			(at 179.07 96.52 0)
+			(effects
+				(font
+					(size 1.27 1.27)
+				)
+				(hide yes)
+			)
+		)
+		(property "Datasheet" "~"
+			(at 179.07 96.52 0)
+			(effects
+				(font
+					(size 1.27 1.27)
+				)
+				(hide yes)
+			)
+		)
+		(property "Description" "Special symbol for telling ERC where power comes from"
+			(at 179.07 96.52 0)
+			(effects
+				(font
+					(size 1.27 1.27)
+				)
+				(hide yes)
+			)
+		)
+		(pin "1"
+		)
+		(instances
+			(project ""
+				(path "/79f480d4-ad37-4b66-a259-96ab4b59ec6d"
+					(reference "#FLG02")
+					(unit 1)
+				)
+			)
+		)
+	)
+	(symbol
 		(lib_id "power:+3V3")
-		(at 170.18 93.98 0)
+		(at 179.07 93.98 0)
 		(unit 1)
 		(exclude_from_sim no)
@@
 		(fields_autoplaced yes)
 		(property "Reference" "#PWR03"
-			(at 170.18 97.79 0)
+			(at 179.07 97.79 0)
 			(effects
 				(font
@@
 		)
 		(property "Value" "+3V3 Buck"
-			(at 170.18 88.9 0)
+			(at 179.07 88.9 0)
 			(effects
 				(font
@@
 		)
 		(property "Footprint" ""
-			(at 170.18 93.98 0)
+			(at 179.07 93.98 0)
 			(effects
 				(font
@@
 		)
 		(property "Datasheet" ""
-			(at 170.18 93.98 0)
+			(at 179.07 93.98 0)
 			(effects
 				(font
@@
 		)
 		(property "Description" "Power symbol creates a global label with name \"+3V3\""
-			(at 170.18 93.98 0)
-			(effects
-				(font
+			(at 179.07 93.98 0)
+			(effects
+				(font

Commit message: ignore production files
Parts:
- C1, C3: LCSC Part # (none) -> C45107
- C2: LCSC Part # (none) -> C15849
- D1: LCSC Part # (none) -> C95400
- J1: LCSC Part # (none) -> C492400
- J2: LCSC Part # (none) -> C124375
- J3: JLC C3096093 -> (none); LCSC Part # (none) -> C3096093
- L1: footprint project_footprints:INDM3225X240N -> Inductor_SMD:L_Chilisin_BMRF00101040; LCSC Part # (none) -> C6364681
- U1: LCSC Part # (none) -> C2681226
Changed lines of the file:
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@@
+			)
+		)
+		(property "LCSC Part #" "C492400"
+			(at 60.96 36.83 0)
+			(effects
+				(font
+					(size 1.27 1.27)
+				)
+				(hide yes)
 			)
 		)
@@
 			)
 		)
+		(property "LCSC Part #" "C124375"
+			(at 63.5 77.47 0)
+			(effects
+				(font
+					(size 1.27 1.27)
+				)
+				(hide yes)
+			)
+		)
 		(pin "1"
 		)
@@
 			)
 		)
-		(property "JLC" "C3096093"
+		(property "LCSC Part #" "C3096093"
 			(at 64.77 49.53 0)
 			(effects
@@
 			)
 		)
+		(property "LCSC Part #" "C2681226"
+			(at 116.84 97.79 0)
+			(effects
+				(font
+					(size 1.27 1.27)
+				)
+				(hide yes)
+			)
+		)
 		(pin "2"
 		)
@@
 			)
 		)
-		(property "Footprint" "project_footprints:INDM3225X240N"
+		(property "Footprint" "Inductor_SMD:L_Chilisin_BMRF00101040"
 			(at 149.86 95.25 0)
 			(effects
@@
 			)
 		)
+		(property "LCSC Part #" "C6364681"
+			(at 149.86 95.25 90)
+			(effects
+				(font
+					(size 1.27 1.27)
+				)
+				(hide yes)
+			)
+		)
 		(pin "1"
 		)
@@
 			)
 		)
-		(property "Description" "C45107"
+		(property "Description" ""
+			(at 163.83 100.33 0)
+			(effects
+				(font
+					(size 1.27 1.27)
+				)
+				(hide yes)
+			)
+		)
+		(property "LCSC Part #" "C45107"
 			(at 163.83 100.33 0)
 			(effects
@@
 			)
 		)
-		(property "Description" "C45107"
+		(property "Description" ""
+			(at 69.85 100.33 0)
+			(effects
+				(font
+					(size 1.27 1.27)
+				)
+				(hide yes)
+			)
+		)
+		(property "LCSC Part #" "C45107"
 			(at 69.85 100.33 0)
 			(effects
@@
 			)
 		)
+		(property "LCSC Part #" "C95400"
+			(at 137.16 100.33 90)
+			(effects
+				(font
+					(size 1.27 1.27)
+				)
+				(hide yes)
+			)
+		)
 		(pin "2"
 		)
@@
 			(at 87.63 100.33 0)
 			(effects
+				(font
+					(size 1.27 1.27)
+				)
+				(hide yes)
+			)
+		)
+		(property "LCSC Part #" "C15849"
+			(at 87.63 100.33 0)
+			(effects
